Commit message: DEX Retargeting

File: autonomy/simulation/Humanoid_Wato/arm_assembly/arm_assembly_fixed.urdf (robot description, URDF)
Before this commit: robot arm_assembly, 22 links, 21 joints
Joints:
- joint cmc_thumb: limit lower=-0.349066 upper=2.094395 effort=100 velocity=100 -> lower=-3.1415 upper=3.1415 effort=100 velocity=100
- joint dip_index: limit lower=-1.570796 upper=0.0 effort=100 velocity=100 -> lower=-3.1415 upper=3.1415 effort=100 velocity=100
- joint dip_middle: limit lower=0.0 upper=1.570796 effort=100 velocity=100 -> lower=-3.1415 upper=3.1415 effort=100 velocity=100
- joint dip_pinky: limit lower=0.0 upper=1.570796 effort=100 velocity=100 -> lower=-3.1415 upper=3.1415 effort=100 velocity=100
- joint dip_ring: limit lower=-1.570796 upper=0.0 effort=100 velocity=100 -> lower=-3.1415 upper=3.1415 effort=100 velocity=100
- joint elbow_flexion_extension: limit lower=-0.349066 upper=3.490659 effort=100 velocity=100 -> lower=-3.1415 upper=3.1415 effort=100 velocity=100
- joint forearm_rotation: limit lower=0.0 upper=3.14 effort=100 velocity=100 -> lower=-3.1415 upper=3.1415 effort=100 velocity=100
- joint ip_thumb: limit lower=0.0 upper=1.570796 effort=100 velocity=100 -> lower=-3.1415 upper=3.1415 effort=100 velocity=100
- joint mcp_index: limit lower=-1.570796 upper=0.0 effort=100 velocity=100 -> lower=-3.1415 upper=3.1415 effort=100 velocity=100
- joint mcp_middle: limit lower=-1.570796 upper=0.0 effort=100 velocity=100 -> lower=-3.1415 upper=3.1415 effort=100 velocity=100
- joint mcp_pinky: limit lower=0.0 upper=1.570796 effort=100 velocity=100 -> lower=-3.1415 upper=3.1415 effort=100 velocity=100
- joint mcp_ring: limit lower=0.0 upper=1.570796 effort=100 velocity=100 -> lower=-3.1415 upper=3.1415 effort=100 velocity=100
- joint mcp_thumb: limit lower=0.785398 upper=2.530727 effort=100 velocity=100 -> lower=-3.1415 upper=3.1415 effort=100 velocity=100
- joint pip_index: limit lower=0.0 upper=1.570796 effort=100 velocity=100 -> lower=-3.1415 upper=3.1415 effort=100 velocity=100
- joint pip_middle: limit lower=0.0 upper=1.570796 effort=100 velocity=100 -> lower=-3.1415 upper=3.1415 effort=100 velocity=100
- joint pip_pinky: limit lower=-1.570796 upper=0.0 effort=100 velocity=100 -> lower=-3.1415 upper=3.1415 effort=100 velocity=100
- joint pip_ring: limit lower=-1.570796 upper=0.0 effort=100 velocity=100 -> lower=-3.1415 upper=3.1415 effort=100 velocity=100
- joint shoulder_abduction_adduction: limit lower=-0.349066 upper=3.490659 effort=100 velocity=100 -> lower=-3.1415 upper=3.1415 effort=100 velocity=100
- joint shoulder_flexion_extension: limit lower=-3.14 upper=3.14 effort=10 velocity=10 -> lower=-3.1415 upper=3.1415 effort=10 velocity=10
- joint shoulder_rotation: limit lower=-3.14 upper=3.14 effort=10 velocity=10 -> lower=-3.1415 upper=3.1415 effort=10 velocity=10
- joint wrist_extension: limit lower=-0.959931 upper=0.959931 effort=100 velocity=100 -> lower=-3.1415 upper=3.1415 effort=100 velocity=100
