Commit message: Arm motion

File: autonomy/simulation/Humanoid_Wato/arm_assembly/simple_door.urdf (robot description, URDF)
Before this commit: robot simple_door, 2 links, 1 joints
Links:
- added link push_marker, mass 0.01; visual sphere radius=0.06
- link door_panel: geometry collision box size=0.08 0.9 2.0; visual box size=0.08 0.9 2.0
Joints:
- added joint marker_joint: type fixed, parent door_panel, child push_marker, origin xyz=0 0 0 rpy=0 0 0

Commit message: Arm motion

File: autonomy/simulation/Humanoid_Wato/arm_assembly/simple_door.urdf (robot description, URDF)
Before this commit: robot simple_door, 3 links, 2 joints
Joints:
- joint door_hinge: limit lower=0.0 upper=0.524 effort=50.0 velocity=1.0 -> lower=-0.524 upper=0.524 effort=50.0 velocity=1.0
