Commit message: removing sim

File: autonomy/simulation/Humanoid_Wato/arm_assembly/arm_assembly.urdf (robot description, URDF)
Before this commit: robot arm_assembly, 22 links, 21 joints
Joints:
- joint shoulder_flexion_extension: limit lower=-3.14 upper=3.14 effort=100 velocity=100 -> (none)
- joint shoulder_rotation: limit lower=-3.14 upper=3.14 effort=100 velocity=100 -> (none)
