Commit message: refactor-and-organize-assets-and-folder

File: autonomy/simulation/Humanoid_Wato/arm_assembly/left_arm_assembly.urdf (robot description, URDF)
Before this commit: robot left_arm_assembly, 22 links, 21 joints
Links:
- link left_CMC_THUMB_v1_1: geometry collision mesh filename=meshes/left_arm/left_CMC_THUMB_v1_1.stl scale=0.001 0.001 0.001; visual mesh filename=meshes/left_arm/left_CMC_THUMB_v1_1.stl scale=0.001 0.001 0.001
- link left_DIP_INDEX_v1_1: geometry collision mesh filename=meshes/left_arm/left_DIP_INDEX_v1_1.stl scale=0.001 0.001 0.001; visual mesh filename=meshes/left_arm/left_DIP_INDEX_v1_1.stl scale=0.001 0.001 0.001
- link left_DIP_MIDDLE_v1_1: geometry collision mesh filename=meshes/left_arm/left_DIP_MIDDLE_v1_1.stl scale=0.001 0.001 0.001; visual mesh filename=meshes/left_arm/left_DIP_MIDDLE_v1_1.stl scale=0.001 0.001 0.001
- link left_DIP_PINKY_v1_1: geometry collision mesh filename=meshes/left_arm/left_DIP_PINKY_v1_1.stl scale=0.001 0.001 0.001; visual mesh filename=meshes/left_arm/left_DIP_PINKY_v1_1.stl scale=0.001 0.001 0.001
- link left_DIP_RING_v1_1: geometry collision mesh filename=meshes/left_arm/left_DIP_RING_v1_1.stl scale=0.001 0.001 0.001; visual mesh filename=meshes/left_arm/left_DIP_RING_v1_1.stl scale=0.001 0.001 0.001
- link left_IP_THUMB_v1_1: geometry collision mesh filename=meshes/left_arm/left_IP_THUMB_v1_1.stl scale=0.001 0.001 0.001; visual mesh filename=meshes/left_arm/left_IP_THUMB_v1_1.stl scale=0.001 0.001 0.001
- link left_MCP_INDEX_v1_1: geometry collision mesh filename=meshes/left_arm/left_MCP_INDEX_v1_1.stl scale=0.001 0.001 0.001; visual mesh filename=meshes/left_arm/left_MCP_INDEX_v1_1.stl scale=0.001 0.001 0.001
- link left_MCP_MIDDLE_v1_1: geometry collision mesh filename=meshes/left_arm/left_MCP_MIDDLE_v1_1.stl scale=0.001 0.001 0.001; visual mesh filename=meshes/left_arm/left_MCP_MIDDLE_v1_1.stl scale=0.001 0.001 0.001
- link left_MCP_PINKY_v1_1: geometry collision mesh filename=meshes/left_arm/left_MCP_PINKY_v1_1.stl scale=0.001 0.001 0.001; visual mesh filename=meshes/left_arm/left_MCP_PINKY_v1_1.stl scale=0.001 0.001 0.001
- link left_MCP_RING_v1_1: geometry collision mesh filename=meshes/left_arm/left_MCP_RING_v1_1.stl scale=0.001 0.001 0.001; visual mesh filename=meshes/left_arm/left_MCP_RING_v1_1.stl scale=0.001 0.001 0.001
- link left_MCP_THUMB_v1_1: geometry collision mesh filename=meshes/left_arm/left_MCP_THUMB_v1_1.stl scale=0.001 0.001 0.001; visual mesh filename=meshes/left_arm/left_MCP_THUMB_v1_1.stl scale=0.001 0.001 0.001
- link left_PALM_GAVIN_1DoF_Hinge_v2_1: geometry collision mesh filename=meshes/left_arm/left_PALM_GAVIN_1DoF_Hinge_v2_1.stl scale=0.001 0.001 0.001; visual mesh filename=meshes/left_arm/left_PALM_GAVIN_1DoF_Hinge_v2_1.stl scale=0.001 0.001 0.001
- link left_PIP_INDEX_v1_1: geometry collision mesh filename=meshes/left_arm/left_PIP_INDEX_v1_1.stl scale=0.001 0.001 0.001; visual mesh filename=meshes/left_arm/left_PIP_INDEX_v1_1.stl scale=0.001 0.001 0.001
- link left_PIP_MIDDLE_v1_1: geometry collision mesh filename=meshes/left_arm/left_PIP_MIDDLE_v1_1.stl scale=0.001 0.001 0.001; visual mesh filename=meshes/left_arm/left_PIP_MIDDLE_v1_1.stl scale=0.001 0.001 0.001
- link left_PIP_PINKY_v1_1: geometry collision mesh filename=meshes/left_arm/left_PIP_PINKY_v1_1.stl scale=0.001 0.001 0.001; visual mesh filename=meshes/left_arm/left_PIP_PINKY_v1_1.stl scale=0.001 0.001 0.001
- link left_PIP_RING_v1_1: geometry collision mesh filename=meshes/left_arm/left_PIP_RING_v1_1.stl scale=0.001 0.001 0.001; visual mesh filename=meshes/left_arm/left_PIP_RING_v1_1.stl scale=0.001 0.001 0.001
- link left_base_link: geometry collision mesh filename=meshes/left_arm/left_base_link.stl scale=0.001 0.001 0.001; visual mesh filename=meshes/left_arm/left_base_link.stl scale=0.001 0.001 0.001
- link left_elbow_link_1_v6_1: geometry collision mesh filename=meshes/left_arm/left_elbow_link_1_v6_1.stl scale=0.001 0.001 0.001; visual mesh filename=meshes/left_arm/left_elbow_link_1_v6_1.stl scale=0.001 0.001 0.001
- link left_elbow_link_2_v7_1: geometry collision mesh filename=meshes/left_arm/left_elbow_link_2_v7_1.stl scale=0.001 0.001 0.001; visual mesh filename=meshes/left_arm/left_elbow_link_2_v7_1.stl scale=0.001 0.001 0.001
- link left_forearm_v8_1: geometry collision mesh filename=meshes/left_arm/left_forearm_v8_1.stl scale=0.001 0.001 0.001; visual mesh filename=meshes/left_arm/left_forearm_v8_1.stl scale=0.001 0.001 0.001
- link left_shoulder_link_1_v9_1: geometry collision mesh filename=meshes/left_arm/left_shoulder_link_1_v9_1.stl scale=0.001 0.001 0.001; visual mesh filename=meshes/left_arm/left_shoulder_link_1_v9_1.stl scale=0.001 0.001 0.001
- link left_shoulder_link_2_v4_1: geometry collision mesh filename=meshes/left_arm/left_shoulder_link_2_v4_1.stl scale=0.001 0.001 0.001; visual mesh filename=meshes/left_arm/left_shoulder_link_2_v4_1.stl scale=0.001 0.001 0.001
