Commit message: Updated reward function

File: autonomy/simulation/Humanoid_Wato/wato_bimanual_arm/urdf/armDouble.SLDASM.urdf (robot description, URDF)
Before this commit: robot armDouble.SLDASM, 17 links, 16 joints
Joints:
- joint joint7: limit lower=-3.1415 upper=3.1415 effort=100 velocity=10 -> lower=-0.09 upper=-0.02 effort=100 velocity=10
- joint joint7l: limit lower=-3.1415 upper=3.1415 effort=100 velocity=10 -> lower=-0.09 upper=-0.02 effort=100 velocity=10
- joint joint8: limit lower=-3.1415 upper=3.1415 effort=100 velocity=10 -> lower=0.02 upper=0.09 effort=100 velocity=10
- joint joint8l: limit lower=-3.1415 upper=3.1415 effort=100 velocity=10 -> lower=0.02 upper=0.09 effort=100 velocity=10

Commit message: Updated reward function

File: autonomy/simulation/Humanoid_Wato/wato_bimanual_arm/urdf/armDouble.SLDASM.urdf (robot description, URDF)
Before this commit: robot armDouble.SLDASM, 17 links, 16 joints
Joints:
- joint joint7: limit lower=-0.09 upper=-0.02 effort=100 velocity=10 -> lower=-0.155 upper=-0.082 effort=100 velocity=10
- joint joint7l: limit lower=-0.09 upper=-0.02 effort=100 velocity=10 -> lower=-0.155 upper=-0.082 effort=100 velocity=10
- joint joint8: limit lower=0.02 upper=0.09 effort=100 velocity=10 -> lower=0.082 upper=0.155 effort=100 velocity=10
- joint joint8l: limit lower=0.02 upper=0.09 effort=100 velocity=10 -> lower=0.082 upper=0.155 effort=100 velocity=10
