Commit message: add-proper-calibration

File: autonomy/simulation/Humanoid_Wato/wato_bimanual_arm/urdf/bimanual_arm.urdf (robot description, URDF)
Before this commit: robot bimanual_arm, 17 links, 16 joints
Joints:
- joint joint1: origin xyz=0 0.16355 0.5172 rpy=0 0 0 -> xyz=0 0.16355 0.5172 rpy=0 3.141592653589793 0
- joint joint2: origin xyz=0.0315 0.084 0 rpy=0 0 0 -> xyz=0.0315 0.084 0 rpy=1.5707963267948966 0 0
- joint joint3: origin xyz=-0.017 0.171 0 rpy=0 0 0 -> xyz=-0.017 0.171 0 rpy=0 -1.5707963267948966 0

File: autonomy/simulation/Humanoid_Wato/wato_bimanual_arm/urdf/bimanual_arm_curobo.urdf (robot description, URDF)
Before this commit: robot armDouble.SLDASM, 17 links, 16 joints
Joints:
- joint joint1: origin xyz=0 0.16355 0.5172 rpy=0 0 0 -> xyz=0 0.16355 0.5172 rpy=0 3.141592653589793 0
- joint joint2: origin xyz=0.0315 0.084 0 rpy=0 0 0 -> xyz=0.0315 0.084 0 rpy=1.5707963267948966 0 0
- joint joint3: origin xyz=-0.017 0.171 0 rpy=0 0 0 -> xyz=-0.017 0.171 0 rpy=0 -1.5707963267948966 0
