Commit message: migrate rl to new docker

File: autonomy/simulation/Humanoid_Wato/wato_hand/urdf/hand_urdf.urdf (robot description, URDF)
Before this commit: robot hand_urdf, 21 links, 20 joints
Joints:
- joint MCP_A_1: limit lower=-0.15 upper=0.15 effort=0 velocity=0 -> lower=-0.471239 upper=0.471239 effort=0 velocity=0
- joint MCP_A_2: limit lower=-0.15 upper=0.15 effort=0 velocity=0 -> lower=-0.471239 upper=0.471239 effort=0 velocity=0
- joint MCP_A_3: limit lower=-0.15 upper=0.15 effort=0 velocity=0 -> lower=-0.471239 upper=0.471239 effort=0 velocity=0
- joint MCP_A_4: limit lower=-0.15 upper=0.15 effort=0 velocity=0 -> lower=-0.471239 upper=0.471239 effort=0 velocity=0
