Commit message: [Teleop] migrated scene to new pioneer usd asset, fixed elbow hyperextension

File: autonomy/simulation/Humanoid_Wato/pioneer_bimanual_arm/urdf/pioneer_bimanual_arm.urdf (robot description, URDF)
Before this commit: robot armv2URDF, 17 links, 16 joints
Joints:
- joint joint4l: limit lower=-1.745329 upper=2.312561 effort=0 velocity=0 -> lower=-2.312561 upper=1.745329 effort=0 velocity=0
- joint joint5: origin xyz=0 0.0274999999999994 -0.1074999991972 rpy=0 0 0 -> xyz=0 0.0229999999999994 -0.1074999991972 rpy=0 0 0
- joint joint5l: origin xyz=0.00126373662642563 -0.0230249983943991 -0.169243101839289 rpy=0 0 0 -> xyz=0 -0.0230249983943991 -0.169243101839289 rpy=0 0 0
- joint joint6: origin xyz=0 0.0325 -0.128000000000001 rpy=0 0 0 -> xyz=0 0.037 -0.128000000000001 rpy=0 0 0
- joint joint6l: origin xyz=-0.00126373662644846 -0.0459750016055988 -0.0662568973579128 rpy=0 0 0 -> xyz=-2.28300451460273e-14 -0.0459750016055988 -0.0662568973579128 rpy=0 0 0

Commit message: [Teleop] fix IL dataset correctness, arm dynamics, joint4 limits

File: autonomy/simulation/Humanoid_Wato/pioneer_bimanual_arm/urdf/pioneer_bimanual_arm.urdf (robot description, URDF)
Before this commit: robot armv2URDF, 17 links, 16 joints
Joints:
- joint joint4: limit lower=-2.312561 upper=1.745329 effort=0 velocity=0 -> lower=-1.745329 upper=2.312561 effort=0 velocity=0
