Commit message: Retarget Quest teleop to pioneer_bimanual_arm (#218)
* Add Quest VR teleop for wato_arm_v2 (armWithStand)

Adapts run_quest_bimanual_teleop.py for the new armWithStand.usd
asset: dedicated armWithStand_v2_cfg.py (joint limits/gains/
fingertip geometry re-derived for this asset's different joint
axes, not copied from bimanual), the VR teleop script itself with
a live-tuned stereo RSD455 head camera, a single-arm keyboard
teleop variant for quick bench testing, and a helper script to
open the bare USD scene for visual inspection.

Co-Authored-By: Claude Sonnet 5 <noreply@anthropic.com>

* Tune stereo head camera position/orientation via live feedback

Restored a clean forward-facing gaze (~50deg downward, no roll,
built directly from forward/up vectors rather than composing
rotations) and re-positioned it after several live-tested
attempts at deriving the pose analytically didn't land correctly.
Also added the same stereo RSD455 preview to keyboard_teleop_armv2.py
so camera framing can be checked while driving the arm by hand.

Co-Authored-By: Claude Sonnet 5 <noreply@anthropic.com>

* Fix front/back and left/right axis mapping, add IK diagnostic tooling

Two axis-sign flips in run_quest_armWithStand_teleop.py's Quest-to-world
mapping, found via live headset testing: X was inverted (left/right felt
backwards), then Y was inverted after confirming X/Z were correct
(front/back was still swapped). Also reverted an experimental bent-arm
rest pose after live testing showed it wasn't actually natural-looking,
back to the URDF zero pose.

Added two standalone test scripts to help isolate future direction/motion
issues without needing the headset: task_space_test_armv2.py (drag a cube
with the mouse, same fingertip IK path as the VR script) and
keyboard_teleop_armv2_lightbox.py (keyboard-driven arm in the same
lightbox scene/camera setup used for VR teleop).

Co-Authored-By: Claude Sonnet 5 <noreply@anthropic.com>

* New VR teleop

* Revert unintended edits to run_quest_bimanual_teleop.py

Comment/refactor cleanup on this file was out of scope for the
wato_arm_v2 VR teleop work -- restored to its state before this branch.

* new vr stuff

* act training ramy checkpoint

* openxr removal

* added mono shell to start all teleop processes

* Quest teleop - fixed friction, reduced frame cycle compute time ~3x

* [Teleop] migrated scene to new pioneer usd asset, fixed elbow hyperextension

* cleaned stale files, restructured viewing angles + right wrist cam, rotated lightbox,
    restored default ACTIVE_MODULES

* [Teleop] fix IL dataset correctness, arm dynamics, joint4 limits

* teleop: one Quest driver — armv2 replaces bimanual, not alongside it

run_quest_armv2_teleop.py was added as a parallel driver "replacing"
run_quest_bimanual_teleop.py but the old one was kept. Commit to the
replacement:

- delete run_quest_bimanual_teleop.py (908) + run_quest_bimanual_teleop.sh
- rename run_quest_armv2_teleop.{py,sh} -> run_quest_bimanual_teleop.{py,sh}
- repoint internal name refs (the .sh launcher, container_start_teleop.sh,
  armWithStand_v2_cfg.py comments)

One Quest driver. quest_isaac_teleop/README.md name refs are already correct
after the rename (its internal line-number pointers still describe the old
script and need a follow-up).

Co-Authored-By: Claude Sonnet 5 <noreply@anthropic.com>
Claude-Session: https://claude.ai/code/session_01EtusD8QWFBLpdMUZPpye5B

* teleop: don't commit Table.STEP (CAD source)

table.usd is the runtime artifact Isaac loads; the SolidWorks STEP export it
was converted from doesn't belong in the repo. Nothing references Table.STEP
in code — only a comment, updated to point back at CAD.

Table/ now holds just table.usd.

Co-Authored-By: Claude Sonnet 5 <noreply@anthropic.com>
Claude-Session: https://claude.ai/code/session_01EtusD8QWFBLpdMUZPpye5B

* teleop: fix robot-placement comment (feet on floor, not the table)

The 1.1997m lift plants the stand feet on the floor at z=0; the table (top
~0.7m) is a separate surface the column passes through. Comment said 'rest
on the TABLE top (z=0)' -- wrong on both counts. No code change.

Co-Authored-By: Claude Sonnet 5 <noreply@anthropic.com>
Claude-Session: https://claude.ai/code/session_01EtusD8QWFBLpdMUZPpye5B

* Update .gitignore

* teleop: trim over-long comments added in this branch

Compress the essay-length comment blocks to what's load-bearing: the choice,
the one-line reason not to revert it, and a pointer. Drop measurement tables,
blow-by-blow history, and re-derivations. No code changes.

Also fix the URDF joint4/joint4l limit-swap comment: the pair was already a
proper negate-swap on main, not "identical" -- the swap moves each elbow's
larger travel budget onto its flexion side, and the comment now says that.

Co-Authored-By: Claude Sonnet 5 <noreply@anthropic.com>
Claude-Session: https://claude.ai/code/session_01EtusD8QWFBLpdMUZPpye5B

* teleop: fix stale references after the armv2 -> single-driver rename

- dataset schema + index.html + both .sh headers: run_quest_armv2_teleop.py ->
  run_quest_bimanual_teleop.py (renamed in 43b4a781)
- container_start_teleop.sh: drop the two-driver auto-detect; there is one now
- README + module docstring: _DLS_LAMBDA is 0.1/0.175 (not 0.2/0.35),
  _AXIS_SIGN is [1,1,1] (not [1,-1,1]), actuator tuning lives in
  armWithStand_v2_cfg.py (not bimanual_arm_cfg.py), _QUEST_TO_WORLD is retired
  in favour of the camera-relative mapping, wrist-offset line pointer, .jpg not .png
- schema: robot_type fallback wording, articulation/column-order note

Co-Authored-By: Claude Sonnet 5 <noreply@anthropic.com>
Claude-Session: https://claude.ai/code/session_01EtusD8QWFBLpdMUZPpye5B

* ci: exclude tools/isaac_harness from autopep8

isaac_session_daemon.py imports isaaclab after AppLauncher(args_cli) (Kit must
launch first); autopep8 'fixes' this by hoisting the imports and breaking the
file. Same AppLauncher-before-imports constraint *autonomy/simulation* is
already excluded for.

Co-Authored-By: Claude Sonnet 5 <noreply@anthropic.com>
Claude-Session: https://claude.ai/code/session_01EtusD8QWFBLpdMUZPpye5B

* sim_recorder: drop the empty-dataset-shell auto-rename, keep the clearer error

The _is_empty_dataset_shell() heuristic + init_dataset() auto-rename silently
moved operator-supplied directories ({root} -> {root}.empty-<ts>) as a side
effect of opening a dataset, and changed behaviour for all 5 SimLeRobotRecorder
consumers (only the Quest one is touched/tested here). Revert to open-or-raise;
keep the richer error (Cause: ... + 'delete it and retry'). The rate_limit /
callable-images change is unaffected.

If the auto-recovery is wanted, it's its own humanoid_il PR.

Co-Authored-By: Claude Sonnet 5 <noreply@anthropic.com>
Claude-Session: https://claude.ai/code/session_01EtusD8QWFBLpdMUZPpye5B

---------

Co-authored-by: Ramy Wahib <ramy.wahib99@gmail.com>
Co-authored-by: Claude Sonnet 5 <noreply@anthropic.com>
Co-authored-by: wilsonchenghy <wilsonchenghy@gmail.com>
Co-authored-by: Wilson Cheng <150957380+wilsonchenghy@users.noreply.github.com>

File: autonomy/simulation/Humanoid_Wato/pioneer_bimanual_arm/urdf/pioneer_bimanual_arm.urdf (robot description, URDF)
Before this commit: robot armv2URDF, 17 links, 16 joints
Joints:
- joint joint4: limit lower=-2.312561 upper=1.745329 effort=0 velocity=0 -> lower=-1.745329 upper=2.312561 effort=0 velocity=0
- joint joint4l: limit lower=-1.745329 upper=2.312561 effort=0 velocity=0 -> lower=-2.312561 upper=1.745329 effort=0 velocity=0
- joint joint5: origin xyz=0 0.0274999999999994 -0.1074999991972 rpy=0 0 0 -> xyz=0 0.0229999999999994 -0.1074999991972 rpy=0 0 0
- joint joint5l: origin xyz=0.00126373662642563 -0.0230249983943991 -0.169243101839289 rpy=0 0 0 -> xyz=0 -0.0230249983943991 -0.169243101839289 rpy=0 0 0
- joint joint6: origin xyz=0 0.0325 -0.128000000000001 rpy=0 0 0 -> xyz=0 0.037 -0.128000000000001 rpy=0 0 0
- joint joint6l: origin xyz=-0.00126373662644846 -0.0459750016055988 -0.0662568973579128 rpy=0 0 0 -> xyz=-2.28300451460273e-14 -0.0459750016055988 -0.0662568973579128 rpy=0 0 0
